File: pcb/lisn-pcb/lisn-pcb.kicad_pcb (KiCad board)
At the start: 2 copper layers, 160 x 159 mm, 88 parts, among them J1 Conn_Coaxial, J2 Conn_Coaxial, J3 62409-1, J4 62409-1, J5 62409-1, J6 62409-1, J7 62409-1, J8 62409-1, J9 62409-1

Commit message: Bump to KiCad 8, add BOM info
Other:
- net class Default removed

Commit message: Add bleed resistors
Parts:
- added R43: 47k, Resistor_THT:R_Axial_DIN0414_L11.9mm_D4.5mm_P15.24mm_Horizontal, F.Cu at (132.9, 72.8)
- added R44: 47k, Resistor_THT:R_Axial_DIN0414_L11.9mm_D4.5mm_P15.24mm_Horizontal, F.Cu at (227.2, 72.5)
- moved R1 3.80 mm to (158.2, 79.0)
Routing:
- net /LINE: track 21.1 -> 9.36 mm
- net /NEUTRAL: track 20.3 -> 9.30 mm
- net Net-(C4-Pad1): track 92.1 -> 98.6 mm
- net Net-(C1-Pad1): track 73.0 -> 75.5 mm

Commit message: Use a larger value for the bleed resistors
Parts:
- R43, R44: value 47k -> 1M
Changed lines of the file:
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@@
 			)
 		)
-		(property "Value" "47k"
+		(property "Value" "1M"
 			(at 7.62 3.37 0)
 			(layer "F.Fab")
@@
 			)
 		)
-		(property "MPN" "ROX1SJ47K"
+		(property "MPN" " ROX1SJ1M0"
 			(at 0 0 0)
 			(unlocked yes)
@@
 			)
 		)
-		(property "Manufacturer Part Number 1" "ROX1SJ47K"
-			(at 0 0 0)
-			(unlocked yes)
-			(layer "F.Fab")
-			(hide yes)
-			(effects
-				(font
-					(size 1 1)
-					(thickness 0.15)
-				)
-			)
-		)
-		(property "Price" "1.66"
+		(property "Manufacturer Part Number 1" " ROX1SJ1M0"
+			(at 0 0 0)
+			(unlocked yes)
+			(layer "F.Fab")
+			(hide yes)
+			(effects
+				(font
+					(size 1 1)
+					(thickness 0.15)
+				)
+			)
+		)
+		(property "Price" ".2"
 			(at 0 0 0)
 			(unlocked yes)
@@
 			)
 		)
-		(property "Supplier Part Number 1" " 279-ROX1SJ47K"
+		(property "Supplier Part Number 1" " 279-ROX1SJ1M0"
 			(at 0 0 0)
 			(unlocked yes)
@@
 		(tags "Resistor Axial_DIN0414 series Axial Horizontal pin pitch 15.24mm 2W length 11.9mm diameter 4.5mm")
 		(property "Reference" "R44"
-			(at 7.44 3.3 360)
-			(layer "F.SilkS")
-			(effects
-				(font
-					(size 1 1)
-					(thickness 0.15)
-				)
-			)
-		)
-		(property "Value" "47k"
-			(at 7.62 3.37 360)
+			(at 7.44 3.3 0)
+			(layer "F.SilkS")
+			(effects
+				(font
+					(size 1 1)
+					(thickness 0.15)
+				)
+			)
+		)
+		(property "Value" "1M"
+			(at 7.62 3.37 0)
 			(layer "F.Fab")
 			(effects
@@
 			)
 		)
-		(property "MPN" "ROX1SJ47K"
+		(property "MPN" "ROX1SJ1M0"
 			(at 0 0 180)
 			(unlocked yes)
@@
 			)
 		)
-		(property "Manufacturer Part Number 1" "ROX1SJ47K"
-			(at 0 0 180)
-			(unlocked yes)
-			(layer "F.Fab")
-			(hide yes)
-			(effects
-				(font
-					(size 1 1)
-					(thickness 0.15)
-				)
-			)
-		)
-		(property "Price" "1.66"
+		(property "Manufacturer Part Number 1" "ROX1SJ1M0"
+			(at 0 0 180)
+			(unlocked yes)
+			(layer "F.Fab")
+			(hide yes)
+			(effects
+				(font
+					(size 1 1)
+					(thickness 0.15)
+				)
+			)
+		)
+		(property "Price" ".2"
 			(at 0 0 180)
 			(unlocked yes)
@@
 			)
 		)
-		(property "Supplier Part Number 1" " 279-ROX1SJ47K"
+		(property "Supplier Part Number 1" "279-ROX1SJ1M0"
 			(at 0 0 180)
 			(unlocked yes)
@@
 		)
 		(fp_text user "${REFERENCE}"
-			(at 7.62 0 360)
-			(layer "F.Fab")
-			(effects
+			(at 7.62 0 0)
+			(layer "F.Fab")
+			(effects
